File: First PCB EVER.kicad_sch (KiCad schematic)
At the start: 4 parts, among them U1 ATmega32U4-A

Commit message: A LOT OF WORK
asdf
Parts:
- added C1: C_Small, Capacitor_SMD:C_0805_2012Metric, symbol Device:C_Small
- added C2, C3, C6: 0.1uF, Capacitor_SMD:C_0805_2012Metric, symbol Device:C_Small
- added C4: 10uF, Capacitor_SMD:C_0805_2012Metric, symbol Device:C_Small
- added C5, C7: 22pF, Capacitor_SMD:C_0805_2012Metric, symbol Device:C_Small
- added D1, D2, D3, D4: D_Small, Diode_SMD:D_SOD-123, symbol Device:D_Small
- added F1: 500mA, Fuse:Fuse_1206_3216Metric, symbol Device:Polyfuse
- added MX1, MX2, MX3, MX4: MX-NoLED, MX_Alps_Hybrid:MX-1U, symbol MX_Alps_Hybrid:MX-NoLED
- added R4: 10k, Resistor_SMD:R_0815_2038Metric, symbol Device:R_Small
- added SW1: SW_Push, random-keyboard-parts:SKQG-1155865, symbol Switch:SW_Push
- added USB1: Molex-0548190589, random-keyboard-parts:Molex-0548190589, symbol random-keyboard-parts:Molex-0548190589
- added Y1: 16MHz, Crystal:Crystal_SMD_3225-4Pin_3.2x2.5mm, symbol Device:Crystal_GND24_Small
- R1: footprint (none) -> Resistor_SMD:R_0815_2038Metric
- R2, R3: value R_Small -> 22; footprint (none) -> Resistor_SMD:R_0815_2038Metric
Connections:
- net +5V: now also U1.7 (VBUS), C2.1, C3.1, C4.1, C6.1, F1.2, R4.1
- net GND: now also C1.1, C2.2, C3.2, C4.2, C5.1, C6.2, C7.1, SW1.1, USB1.1 (GND), Y1.2, Y1.4; no longer R2.2, R3.1
- net at U1.13 (~{RESET}): now also R4.2, SW1.2
- net at U1.16 (XTAL2): now also C5.2, Y1.3
- net at U1.17 (XTAL1): now also C7.2, Y1.1
- net ROW0: now reaches U1.27 (PD7)
- net ROW0: now also D1.1 (K), D2.1 (K)
- net COL1: now reaches U1.28 (PB4)
- net COL1: now also MX2.1 (COL), MX4.1 (COL)
- net COL0: now reaches U1.29 (PB5)
- net COL0: now also MX1.1 (COL), MX3.1 (COL)
- net ROW1: now reaches U1.30 (PB6)
- net ROW1: now also D3.1 (K), D4.1 (K)
- net at U1.6 (UCAP): now also C1.2
- new net: D4.2 (A), MX4.2 (ROW)
- new net: D3.2 (A), MX3.2 (ROW)
- new net: D2.2 (A), MX2.2 (ROW)
- new net: D1.2 (A), MX1.2 (ROW)
- new net D+: R2.2, USB1.3 (D+)
- new net D-: R3.1, USB1.4 (D-)
- new net VCC: F1.1, USB1.5 (VBUS)
Other:
- moved on the sheet: R1, R2, R3, U1
